File: Hardware/T1000/T1000.kicad_pcb (KiCad board)
At the start: 4 copper layers, 103 parts, among them J1 USB_C_Receptacle_USB2.0, J2 SOICbite, J3 XT30, J4 Nichrome, Q1 IRLML0060TRPBF, U1 LT3120JV-PBF, U2 RP2040, U3 W25Q128JVS, U4 LTC4419, U5 MAX-M10S, U6 MS5607-02BA, U7 LT6703CDC-3, U8 MAX77857, U9 XBee_SMT, Y1 445I23D12M00000

Commit message: bringing it together, also managed to crash Kicad so this commit can be considered under duress in a court of law
Parts:
- removed U5: MAX-M10S, RF_GPS:ublox_MAX
- added C43: 100nF, Capacitor_SMD:C_0603_1608Metric_Pad1.08x0.95mm_HandSolder, F.Cu at (147.8, 52.7)
- added R30: 0, Resistor_SMD:R_0603_1608Metric_Pad0.98x0.95mm_HandSolder, F.Cu at (154.0, 58.9)
- added R31: 0, Resistor_SMD:R_0603_1608Metric_Pad0.98x0.95mm_HandSolder, F.Cu at (149.9, 58.9)
- added U10: ~, Terminator_Lib:MIA-M10Q, F.Cu at (151.2, 55.5)
- added Y2: 32.768k, Crystal:Crystal_SMD_3215-2Pin_3.2x1.5mm, F.Cu at (150.9, 51.7)
- C30, C35, C36, C37, J1, R14, U9: moved to B.Cu
- R1: value DNP -> 1k
- moved R7 136.3 mm to (56.9, 152.8), turned to 180 degrees
- moved AE1 127.1 mm to (164.3, 54.0)
- moved Q1 118.3 mm to (56.6, 157.0)
- moved J2 102.6 mm to (132.7, 38.3), turned to 180 degrees
- moved C7 102.6 mm to (131.5, 50.1)
- moved U3 102.6 mm to (120.7, 56.1)
- moved C1 102.6 mm to (131.5, 49.0)
- moved C10 102.6 mm to (127.3, 47.0)
- moved C12 102.6 mm to (124.6, 47.5)
- moved C13 102.6 mm to (124.6, 49.5)
- moved C14 102.6 mm to (129.1, 47.0)
- moved C15 102.6 mm to (124.0, 44.2)
- moved C4 102.6 mm to (124.6, 48.5)
- moved C5 102.6 mm to (124.6, 50.5)
- moved C6 102.6 mm to (126.3, 47.0)
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Connections:
- R21 pad 1: /GPS_RX -> /GPS_TX
- R22 pad 1: /GPS_TX -> /GPS_RX
- U2 pad 15: unconnected-(U2-GPIO12-Pad15) -> /GPS_RX
- U2 pad 16: unconnected-(U2-GPIO13-Pad16) -> /GPS_TX
Routing:
- net /GPS_TX: track 0.00 -> 17.0 mm
- net /GPS_RX: track 0.00 -> 16.8 mm
- net Net-(U2-RUN): track 0.00 -> 13.1 mm
- net Net-(J2-Pin_3): track 0.00 -> 11.8 mm
- net Net-(J2-Pin_2): track 0.00 -> 11.4 mm
- net Net-(U2-XIN): track 0.00 -> 9.28 mm
- net /SDA: track 0.00 -> 8.49 mm
- net Net-(B2-Pad2): track 0.00 -> 7.45 mm
- net GND: track 12.1 -> 19.5 mm
- net +VDC: track 0.00 -> 7.07 mm
- net Net-(U7-IN+): track 0.00 -> 6.77 mm, vias 0 -> 2
- net /SCL: track 0.00 -> 5.45 mm
- net /LVC: track 0.40 -> 5.47 mm
- net Net-(U1-BST3): track 0.00 -> 4.97 mm
- net /USB_D+: track 0.00 -> 4.85 mm
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- added copper zone on F.Cu, net +BATT
- added copper zone on F.Cu, net VBUS
