File: Hardware/T1000/Digital/radio.kicad_sch (KiCad schematic)
At the start: 20 parts, among them J6 Conn_Coaxial, U10 BGS12WN6E6327, U9 SX1262IMLTRT

Commit message: V0 changes before order
Other:
- note added: "Reference design used can be found at: https://www.semtech.com/products/wireless-rf/lora-connect/sx1262"
- company: (none) -> UMDBPP
- title: (none) -> T1000 - LoRa Radio
Changed lines of the file:
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@@
 	(paper "USLetter")
 	(title_block
+		(title "T1000 - LoRa Radio")
 		(date "2024-09-06")
+		(rev "V0")
+		(company "UMDBPP")
+		(comment 1 "Michael Shipman")
+		(comment 2 "ENEE499L")
 	)
 	(junction
@@
 		)
 	)
+	(text "Reference design used can be found at:\nhttps://www.semtech.com/products/wireless-rf/lora-connect/sx1262"
+		(exclude_from_sim no)
+		(at 16.51 194.31 0)
+		(effects
+			(font
+				(size 2.54 2.54)
+			)
+			(justify left)
+		)
+	)
