File: Hardware/T1000/Digital/Digital.kicad_pcb (KiCad board)
At the start: 6 copper layers, 48 x 40 mm, 91 parts, among them J1 Conn_01x02_Pin, J2 Conn_01x06_Socket, J3 Conn_01x04_Pin, J4 FTSH-107-01-L-DV-K-A, J5 USB_C_Receptacle_USB2.0, J6 Conn_Coaxial, SW1 SW_SPDT, SW2 SW_SPDT, U1 MS5607-02BA, U10 BGS12WN6E6327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

Commit message: V0 changes before order
Parts:
- added C35: 10uF, Capacitor_SMD:C_0805_2012Metric, F.Cu at (161.9, 149.3)
- added H1: MountingHole, MountingHole:MountingHole_2.2mm_M2, F.Cu at (187.2, 133.8)
- added H2: MountingHole, MountingHole:MountingHole_2.2mm_M2, F.Cu at (170.9, 150.2)
- added R23: ??, Resistor_SMD:R_0402_1005Metric, F.Cu at (156.9, 139.9)
- added R24: 51k, Resistor_SMD:R_0402_1005Metric, F.Cu at (170.5, 126.7)
- added REF**: BalloonArt_Mask, BPP_Lib:BalloonArt_Mask, F.Cu at (181.7, 124.6)
- added U11: LTC3306CACBZ-R7, BPP_Lib:CB-6-19_ADI, F.Cu at (158.3, 146.5)
- C18, C22: value 10uF -> 1uF; footprint Capacitor_SMD:C_0805_2012Metric -> Capacitor_SMD:C_0603_1608Metric
- C19: value 2.2pF -> 10uF; footprint Capacitor_SMD:C_0402_1005Metric -> Capacitor_SMD:C_0805_2012Metric
- C20: value 15uF -> 2.2pF; footprint Capacitor_SMD:C_1206_3216Metric -> Capacitor_SMD:C_0402_1005Metric
- C21: value 1uF -> 15uF; footprint Capacitor_SMD:C_0603_1608Metric -> Capacitor_SMD:C_1206_3216Metric
- J1: footprint Connector_PinHeader_1.00mm:PinHeader_1x02_P1.00mm_Vertical -> Connector_PinHeader_2.54mm:PinHeader_1x02_P2.54mm_Vertical
- R13: value 649k -> ??k; moved to B.Cu
- R14: value 294k -> 649k
- R15: value ?? -> 294k
- R16: value 100k -> ??
- R17: value 113k -> 100k
- R18: value 0 -> 113k
- R19: value 100k -> 0
- R20: value ?? -> 100k
- U7: value LTC4065EDC-TRMPBF -> LM66100DCKR; footprint BPP_Lib:DFN-6_DC_LIT -> Package_TO_SOT_SMD:SOT-363_SC-70-6
- U8: value LTC3306CACBZ-R7 -> LTC4065EDC-TRMPBF; footprint BPP_Lib:CB-6-19_ADI -> BPP_Lib:DFN-6_DC_LIT
- moved C21 12.8 mm to (166.8, 148.2), turned to -90 degrees
- moved C18 11.1 mm to (162.0, 137.9)
- moved C20 10.2 mm to (156.2, 145.1), turned to 0 degrees
- moved R18 6.92 mm to (158.2, 143.9), turned to 0 degrees
- moved C22 6.58 mm to (161.7, 141.3), turned to 0 degrees
- moved R20 5.98 mm to (162.1, 142.6), turned to 180 degrees
- moved L2 5.63 mm to (163.1, 145.8)
- moved R11 5.50 mm to (162.1, 143.6), turned to 0 degrees
- moved R17 5.25 mm to (160.0, 143.9), turned to 90 degrees
- moved R13 5.03 mm to (159.9, 138.5)
- moved R19 4.79 mm to (162.2, 140.0), turned to 180 degrees
- moved D2 4.57 mm to (153.8, 140.3), turned to 180 degrees
- moved C19 3.71 mm to (156.1, 147.4), turned to -90 degrees
- moved R16 3.55 mm to (153.3, 141.7), turned to 180 degrees
- moved R14 3.36 mm to (158.2, 145.0)
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Connections:
- C18 pad 1: +BATT -> VBUS
- C19 pad 1: Net-(C19-Pad1) -> +BATT
- C19 pad 2: Net-(U8-FB) -> GND
- C20 pad 1: +1V8 -> Net-(C20-Pad1)
- C20 pad 2: GND -> Net-(U11-FB)
- C21 pad 1: VBUS -> +1V8
- C21 pad 2: Net-(C21-Pad2) -> GND
- C22 pad 1: Net-(C19-Pad1) -> Net-(U7-Vout)
- C22 pad 2: GND -> Net-(C22-Pad2)
- C23 pad 1: Net-(C19-Pad1) -> Net-(C20-Pad1)
- L1 pad 1: Net-(U8-SW) -> Net-(U11-SW)
- L1 pad 2: Net-(C19-Pad1) -> Net-(C20-Pad1)
- L2 pad 1: Net-(C19-Pad1) -> Net-(C20-Pad1)
- R11 pad 1: Net-(C19-Pad1) -> Net-(C20-Pad1)
- R13 pad 1: +BATT -> Net-(U7-Vout)
- R13 pad 2: Net-(U8-EN) -> Net-(U7-ST)
- R14 pad 1: Net-(C19-Pad1) -> +BATT
- R14 pad 2: Net-(U8-FB) -> Net-(U11-EN)
- R15 pad 1: VBUS -> Net-(C20-Pad1)
- R15 pad 2: Net-(D2-A) -> Net-(U11-FB)
- R16 pad 1: Net-(U8-EN) -> Net-(U7-Vout)
- R16 pad 2: GND -> Net-(D2-A)
- R17 pad 1: Net-(U8-FB) -> Net-(U11-EN)
- R18 pad 1: Net-(C21-Pad2) -> Net-(U11-FB)
- R19 pad 1: Net-(U8-PGOOD) -> Net-(C22-Pad2)
- R19 pad 2: +1V8 -> GND
- R20 pad 1: Net-(U7-PROG) -> Net-(U11-PGOOD)
- R20 pad 2: GND -> +1V8
- TP3 pad 1: Net-(U8-PGOOD) -> Net-(U11-PGOOD)
- U7 pad 1: GND -> VBUS
- U7 pad 2: Net-(D2-K) -> GND
- U7 pad 3: +BATT -> Net-(U7-Vout)
- U7 pad 4: VBUS -> unconnected-(U7-NC-Pad4)
- U7 pad 5: GND -> Net-(U7-ST)
- U7 pad 6: Net-(U7-PROG) -> Net-(U7-Vout)
Routing:
- net Net-(C19-Pad1): track 20.2 -> 0.00 mm, vias 2 -> 0
- net GND: track 88.0 -> 106.2 mm, vias 84 -> 217
- net Net-(C20-Pad1): track 0.00 -> 15.7 mm, vias 0 -> 2
- net Net-(U7-Vout): track 0.00 -> 14.6 mm, vias 0 -> 3
- net +1V8: track 13.0 -> 4.42 mm, vias 2 -> 0
- net VBUS: track 36.5 -> 27.9 mm, vias 7 -> 6
- net Net-(U11-PGOOD): track 0.00 -> 7.55 mm, vias 0 -> 2
- net Net-(U8-FB): track 5.62 -> 0.00 mm
- net Net-(U6-ST): track 9.26 -> 5.44 mm
- net Net-(U11-FB): track 0.00 -> 3.75 mm
- net Net-(U8-PGOOD): track 3.75 -> 0.00 mm
- net Net-(U8-EN): track 3.31 -> 0.00 mm
- net Net-(U11-EN): track 0.00 -> 2.95 mm
- net VDD: track 68.1 -> 71.0 mm
- net Net-(U8-PROG): track 0.00 -> 2.21 mm
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- removed copper zone on F.Cu, net +BATT
- removed copper zone on In2.Cu, net +BATT
Other:
- board text added: "Michael Shipman V0.0 9/11/2024"
- board text added: "Terminator Logic Board"

Commit message: started STM32 package change (T1001)
Parts:
- removed C10: 1uF, Capacitor_SMD:C_0603_1608Metric
- removed J4: FTSH-107-01-L-DV-K-A, Connector_Samtec:CON14_2X7_DUK_FTSH_SAI-L
- removed U3: STM32L422TBYx, Package_CSP:ST_WLCSP-36_2.58x3.07mm_Layout6x6_P0.4mm
- added J7: Conn_01x05_Pin, Connector_PinHeader_2.54mm:PinHeader_1x05_P2.54mm_Vertical, F.Cu at (165.0, 116.3)
- added R25: 10k, Resistor_SMD:R_0402_1005Metric, F.Cu at (157.0, 121.3)
- added U12: STM32L422KBUx, Package_DFN_QFN:QFN-32-1EP_5x5mm_P0.5mm_EP3.45x3.45mm, F.Cu at (169.9, 133.2)
- J3: value Conn_01x04_Pin -> Conn_01x05_Pin; footprint Connector_PinHeader_2.54mm:PinHeader_1x04_P2.54mm_Vertical -> Connector_PinHeader_2.54mm:PinHeader_1x05_P2.54mm_Vertical
- R13: value ??k -> 10k
- R16: value ?? -> 600
- R23: value ?? -> 6.8k
- R8: value 100 -> 0
- Y2: value Crystal_Small -> 32.768k
- moved R8 26.1 mm to (141.6, 135.1)
- moved C11 20.9 mm to (158.3, 115.7)
- moved C8 10.8 mm to (178.7, 130.1), turned to 90 degrees
- moved J3 9.78 mm to (161.0, 116.3), turned to 0 degrees
- moved C4 8.86 mm to (173.4, 139.8), turned to 180 degrees
- moved C3 7.78 mm to (177.4, 129.5)
- moved C9 7.07 mm to (178.5, 133.2), turned to 0 degrees
- moved R2 6.51 mm to (182.4, 130.6)
- moved C15 6.46 mm to (168.1, 115.9), turned to 0 degrees
- moved X1 6.41 mm to (175.2, 129.8), turned to -90 degrees
- moved L5 6.39 mm to (178.5, 132.2), turned to 180 degrees
- moved C12 5.36 mm to (174.9, 136.2), turned to 90 degrees
- moved R1 5.32 mm to (148.0, 127.4)
- moved C7 5.00 mm to (166.2, 130.5), turned to 90 degrees
- moved Y2 3.77 mm to (176.6, 136.1), turned to -90 degrees
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Connections:
- D1 pad 1: /USB_D- -> /USB_D+
- D1 pad 3: /USB_D+ -> /USB_D-
- J2 pad 5: /COMP2_INP -> /PA3_ADC
- J3 pad 2: /PB10 -> /PA15
- J3 pad 3: /PA8 -> /PA6
- J3 pad 4: VDD -> /PA8
- J5 pad A6: Net-(D1-L2-Pad4) -> Net-(D1-L1-Pad6)
- J5 pad A7: Net-(D1-L1-Pad6) -> Net-(D1-L2-Pad4)
- J5 pad B6: Net-(D1-L2-Pad4) -> Net-(D1-L1-Pad6)
- J5 pad B7: Net-(D1-L1-Pad6) -> Net-(D1-L2-Pad4)
- R5 pad 2: Net-(SW2-C) -> Net-(SW2-B)
- R8 pad 1: Net-(J4-Pin_11) -> VDD
- R8 pad 2: GND -> Net-(U12-PB5)
- SW1 pad 2: /T_NRST -> GND
- SW1 pad 3: GND -> /T_NRST
- U9 pad 13: /PA9 -> /RADIO_DIO1
- U9 pad 14: /PB3 -> /RADIO_BUSY
Routing:
- net /T_NRST: track 75.1 -> 34.5 mm, vias 8 -> 4
- net /PB3: track 38.7 -> 0.00 mm, vias 4 -> 0
- net /TIM1_CH3: track 35.7 -> 0.00 mm, vias 2 -> 0
- net /PA9: track 31.9 -> 0.00 mm, vias 4 -> 0
- net Net-(SW2-B): track 30.4 -> 0.00 mm, vias 2 -> 0
- net /COMP2_INP: track 29.3 -> 0.00 mm, vias 4 -> 0
- net /PA3_ADC: track 0.00 -> 26.3 mm, vias 0 -> 2
- net /RADIO_BUSY: track 0.00 -> 23.7 mm, vias 0 -> 2
- net /RADIO_DIO1: track 0.00 -> 17.6 mm, vias 0 -> 3
- net /PB10: track 17.5 -> 0.00 mm, vias 1 -> 0
- net /PA8: track 17.0 -> 0.98 mm
- net /SPI1_MISO: track 45.0 -> 29.8 mm, vias 3 -> 2
- net /FRAM_NSS: track 19.5 -> 6.25 mm, vias 2 -> 1
- net /I2C1_SDA: track 26.8 -> 14.0 mm, vias 3 -> 2
- net /I2C1_SCL: track 24.9 -> 12.5 mm, vias 2 -> 0
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
Commit message: ordered T1001
Parts:
- removed R5: 10k, Resistor_SMD:R_0402_1005Metric
- removed R8: 0, Resistor_SMD:R_0402_1005Metric
- BT1: footprint Connector_JST:JST_PH_S2B-PH-K_1x02_P2.00mm_Horizontal -> Connector_PinHeader_2.54mm:PinHeader_1x02_P2.54mm_Vertical
- moved R1 10.6 mm to (158.3, 125.0), turned to 90 degrees
- moved R2 1.77 mm to (181.2, 129.3)
- moved C15 1.50 mm to (168.8, 117.2), turned to 90 degrees
- moved R24 1.12 mm to (171.0, 125.7)
- moved R9 0.60 mm to (160.5, 131.7)
- turned BT1 to 180 degrees
Connections:
- SW2 pad 2: Net-(SW2-B) -> GND
- U12 pad 28: Net-(U12-PB5) -> VDD
Routing:
- net /TIM1_CH3: track 0.00 -> 30.2 mm, vias 0 -> 1
- net /T_NRST: track 34.5 -> 64.0 mm, vias 4 -> 9
- net Net-(U12-PH3): track 0.00 -> 27.3 mm, vias 0 -> 2
- net /PA15: track 0.00 -> 24.4 mm, vias 0 -> 1
- net /FRAM_NSS: track 6.25 -> 25.6 mm, vias 1 -> 4
- net /PA6: track 0.00 -> 17.8 mm, vias 0 -> 2
- net /RADIO_DIO1: track 17.6 -> 35.0 mm, vias 3 -> 4
- net /I2C1_SCL: track 12.5 -> 29.2 mm, vias 0 -> 2
- net /I2C1_SDA: track 14.0 -> 30.7 mm, vias 2 -> 3
- net /RADIO_NSS: track 22.0 -> 38.0 mm, vias 2 -> 4
- net /SPI1_MOSI: track 29.1 -> 43.0 mm, vias 3 -> 5
- net /SPI1_SCK: track 30.9 -> 42.0 mm, vias 4 -> 5
- net /PA8: track 0.98 -> 11.5 mm
- net Net-(SW1-A): track 0.00 -> 6.80 mm
- net /SPI1_MISO: track 29.8 -> 35.5 mm, vias 2 -> 3
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Other:
- board text added: "+"
- board text added: "BOOT0"
- board text added: "GND"
- board text added: "Michael Shipman V0.0 10/08/2024"
- board text added: "RST"
- board text added: "SWCLK"
- board text added: "SWDIO"
- board text added: "Vdd"
- board text removed: "Michael Shipman V0.0 9/11/2024"
