File: Hardware/T1000/Digital/power.kicad_sch (KiCad schematic)
At the start: 30 parts, among them U11 LTC3306CACBZ-R7, U5 MIC5504-3.3YM5, U6 LM66200DRLR, U7 LM66100DCKR, U8 LTC4065EDC-TRMPBF

Commit message: ordered T1001
Parts:
- BT1: footprint Connector_JST:JST_PH_S2B-PH-K_1x02_P2.00mm_Horizontal -> Connector_PinHeader_2.54mm:PinHeader_1x02_P2.54mm_Vertical
Changed lines of the file:
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@@
 			)
 		)
-		(property "Footprint" "Connector_JST:JST_PH_S2B-PH-K_1x02_P2.00mm_Horizontal"
+		(property "Footprint" "Connector_PinHeader_2.54mm:PinHeader_1x02_P2.54mm_Vertical"
 			(at 100.33 114.046 90)
 			(effects
